Commit message: Atualizando para receber casos de teste

File: model/test_axis/furuta_test_h.xacro (robot description, xacro)
@@ -22,10 +22,9 @@
                 <inertial pos="0 0 0" mass="${mass}" diaginertia="${X_Y_Inertia} ${X_Y_Inertia} ${Z_Inertia}"/>
                 <joint name="motor" pos="0 0 -1.5" type="hinge" axis="1 0 0"/>
-                <body name="haste_vertical" pos="-1.5 0 1.71" axisangle="0 1 0 90">
+                <!-- <body name="haste_vertical" pos="-1.5 0 1.71" axisangle="0 1 0 90">
                     <geom name="haste_vertical_geom" type="cylinder" rgba="0 0 1 1" size=".2 1.5" mass="10"/>
                     <inertial pos="0 0 0" mass="${mass}" diaginertia="${X_Y_Inertia} ${X_Y_Inertia} ${Z_Inertia}"/>
                     <joint name="conector" pos="0 0 1.5" limited="false" type="hinge" axis="1 0 0"/>
-                    <!-- <joint name="motor_vertical" pos="0 0 1.5" type="hinge" axis="1 0 0"/> -->
-                </body>
+                </body> -->
             </body>
         </body>

File: model/test_axis/furuta_test_v.xacro (robot description, xacro)
@@ -21,10 +21,10 @@
                 <geom name="haste_horizontal_geom" type="cylinder" rgba="0 1 0 1" size=".2 1.5" mass="10"/>
                 <inertial pos="0 0 0" mass="${mass}" diaginertia="${X_Y_Inertia} ${X_Y_Inertia} ${Z_Inertia}"/>
-                <joint name="motor" pos="0 0 -1.5" type="hinge" axis="1 0 0"/>
+                <!-- <joint name="motor" pos="0 0 -1.5" type="hinge" axis="1 0 0"/> -->
                 <body name="haste_vertical" pos="-1.5 0 1.71" axisangle="0 1 0 90">
                     <geom name="haste_vertical_geom" type="cylinder" rgba="0 0 1 1" size=".2 1.5" mass="10"/>
                     <inertial pos="0 0 0" mass="${mass}" diaginertia="${X_Y_Inertia} ${X_Y_Inertia} ${Z_Inertia}"/>
-                    <joint name="conector" pos="0 0 1.5" limited="false" type="hinge" axis="1 0 0"/>
-                    <!-- <joint name="motor_vertical" pos="0 0 1.5" type="hinge" axis="1 0 0"/> -->
+                    <!-- <joint name="conector" pos="0 0 1.5" limited="false" type="hinge" axis="1 0 0"/> -->
+                    <joint name="motor_vertical" pos="0 0 1.5" type="hinge" axis="1 0 0"/>
                 </body>
             </body>
@@ -32,6 +32,6 @@
     </worldbody>
     <actuator>
-        <motor name="motor"  joint="motor"/>
-        <!-- <motor name="motor_vertical"  joint="motor_vertical"/> -->
+        <!-- <motor name="motor"  joint="motor"/> -->
+        <motor name="motor_vertical"  joint="motor_vertical"/>
         <!-- <motor name="conector"  joint="conector"/> -->
     </actuator>
