Commit message: atu

File: model/furuta.xacro (robot description, xacro)
@@ -25,6 +25,6 @@
                     <geom name="haste_vertical_geom" type="cylinder" rgba="0 0 1 1" size=".2 1.5" mass="10"/>
                     <inertial pos="0 0 0" mass="${mass}" diaginertia="${X_Y_Inertia} ${X_Y_Inertia} ${Z_Inertia}"/>
-                    <joint name="conector" pos="0 0 1.5" limited="false" type="hinge" axis="1 0 0"/>
-                    <!-- <joint name="motor_vertical" pos="0 0 1.5" type="hinge" axis="1 0 0"/> -->
+                    <!-- <joint name="conector" pos="0 0 1.5" limited="false" type="hinge" axis="1 0 0"/> -->
+                    <joint name="motor_vertical" pos="0 0 1.5" type="hinge" axis="1 0 0"/>
                 </body>
             </body>
@@ -33,5 +33,5 @@
     <actuator>
         <motor name="motor"  joint="motor"/>
-        <!-- <motor name="motor_vertical"  joint="motor_vertical"/> -->
+        <motor name="motor_vertical"  joint="motor_vertical"/>
         <!-- <motor name="conector"  joint="conector"/> -->
     </actuator>

Commit message: atu

File: model/furuta.xacro (robot description, xacro)
@@ -1,4 +1,4 @@
 <mujoco xmlns:xacro="http://www.ros.org/wiki/xacro" model="furuta_pendulum">
-    <xacro:property name="mass" value="10" />
+    <xacro:property name="mass" value="1" />
     <xacro:property name="r"    value="0.2" />
     <xacro:property name="h"    value="1.5" />
@@ -10,5 +10,5 @@
         <material name="MatPlane" reflectance="0.5" shininess="1" specular="1" texrepeat="2 2" texture="texplane"/>
     </asset>
-    <option integrator="RK4" iterations="50" solver="PGS" timestep="0.003" >
+    <option integrator="Euler" iterations="50" solver="PGS" timestep="0.003" >
         <!-- <flags solverstat="enable" energy="enable"/>-->
     </option>

Commit message: Atu

File: model/furuta.xacro (robot description, xacro)
@@ -25,5 +25,4 @@
                     <geom name="haste_vertical_geom" type="cylinder" rgba="0 0 1 1" size=".2 1.5" mass="10"/>
                     <inertial pos="0 0 0" mass="${mass}" diaginertia="${X_Y_Inertia} ${X_Y_Inertia} ${Z_Inertia}"/>
-                    <!-- <joint name="conector" pos="0 0 1.5" limited="false" type="hinge" axis="1 0 0"/> -->
                     <joint name="motor_vertical" pos="0 0 1.5" type="hinge" axis="1 0 0"/>
                 </body>
